File: Audio_PA.sch (KiCad schematic (older format))
At the start: 0 parts

Commit message: Electric circuit Ver_1
Parts:
- added C? (x2): 1uF, symbol C
- added C?: 330pF, symbol C
- added C?: 47uF, symbol CP1
- added C?: 10nF, symbol C
- added C? (x3): 100nF, symbol C
- added C?: 100uF, symbol CP1
- added C? (x2): 18pF, symbol C
- added C? (x2): 1000uF, symbol CP1
- added D? (x2): 15V, symbol D_Zener
- added D? (x2): 1N4148, symbol D
- added F? (x2): 3A, symbol Fuse
- added P?: Audio_In, symbol CONN_01X02
- added P?: -45VDC, symbol CONN_01X01
- added P?: Audio_Out, symbol CONN_01X02
- added P?: +45VDC, symbol CONN_01X01
- added Q? (x4): BCM856DS, symbol BCM856DS
- added Q? (x3): MJE350, symbol MJE350
- added Q? (x3): MJE340, symbol MJE340
- added Q?: BD139, symbol BD139
- added Q?: 2N3904, symbol Q_NPN_EBC
- added Q?: 2N3906, symbol Q_PNP_EBC
- added Q?: Q_NMOS_GDS, symbol Q_NMOS_GDS
- added Q?: Q_PMOS_GDS, symbol Q_PMOS_GDS
- added R?: 47K, symbol R
- added R?: 2K2, symbol R
- added R? (x3): 1K, symbol R
- added R? (x3): 470R, symbol R
- added R? (x4): 10K, symbol R
- added R? (x3): 100R, symbol R
- added R?: 27K, symbol R
- added R? (x2): 3K9, symbol R
- added R?: 10R, symbol R
- added R? (x4): R, symbol R
- added R? (x2): 0R33, symbol R
- added R? (x2): 330R, symbol R
- added RV?: 100R, symbol POT_TRIM
- added RV?: 1K, symbol POT_TRIM
Connections:
- new net: C?.1, C?.1, P?.1 (P1)
- new net: C?.2, C?.2, R?.1, R?.2
- new net: C?.1, Q?.2 (B), R?.1
- new net: Q?.1 (E), RV?.1
- new net: C?.2, Q?.3 (B), Q?.6 (C), R?.1
- new net: C?.1, Q?.3 (B), Q?.3 (C), R?.1
- new net: Q?.4 (E), RV?.3
- new net: Q?.5 (B), R?.1, R?.2
- new net: Q?.3 (C), RV?.2
- new net: C?.1, Q?.1 (E), Q?.1 (E), R?.1, R?.1, R?.1
- new net: Q?.2 (B), R?.1
- new net: Q?.5 (B), Q?.6 (C), R?.1
- new net: Q?.4 (E), R?.2, R?.2
- new net: C?.2, R?.1, R?.2
- new net: Q?.1 (E), R?.2 (x2)
- new net: Q?.2 (C), Q?.3 (B), Q?.3 (B), R?.1
- new net: C?.1, D?.1 (K), Q?.2 (C), Q?.2 (C), R?.1, R?.1
- new net: Q?.1 (E), Q?.1 (E), R?.1
- new net: C?.2, Q?.2 (C), R?.2
- new net: C?.1, C?.2, D?.2 (A), Q?.1 (E), Q?.2 (C), R?.1, R?.2
- new net: C?.1, C?.1, C?.1, R?.2
- new net: C?.1, D?.1 (K), D?.2 (A), P?.1 (P1), Q?.1 (E), Q?.1 (E), R?.1, R?.1, R?.1, R?.2, R?.2
- new net: Q?.1 (E), R?.2, R?.2, R?.2
- new net: F?.1, P?.1 (P1) (x2)
- new net: F?.2, Q?.2 (C), Q?.3 (S), R?.1
- new net: C?.2, R?.1
- new net: Q?.3 (B), R?.2, RV?.3
- new net: R?.1, RV?.1, RV?.2
- new net: D?.2 (A), Q?.1 (G), R?.2
- new net: D?.1 (K), Q?.1 (G), R?.2
- new net: D?.1 (K), Q?.3 (C)
- new net: D?.2 (A), Q?.3 (C)
- new net: Q?.2 (B), R?.1, R?.2 (x2)
- new net: Q?.3 (S), R?.1, R?.1
- new net: Q?.2 (D), R?.2, R?.2
- new net: F?.2, Q?.2 (C), Q?.2 (D), R?.1
- new net: C?.1, Q?.3 (B), R?.2
- new net: C?.2, Q?.3 (B), R?.2
- new net Earth: C?.1, C?.2, C?.2, C?.2, C?.2, P?.2 (P2), P?.2 (P2), R?.2, R?.2, R?.2

Commit message: Electric circuit Ver_1.1
Parts:
- removed R? (x2): R, symbol R
- added R23: 82R, symbol R
- added R24: 33R, symbol R
- added RV3, RV4: 50, symbol POT_TRIM
- Q12: renamed from Q?; value Q_NMOS_GDS -> IRFP240
- Q13: renamed from Q?; value Q_PMOS_GDS -> IRFP9240
- R21: renamed from R?; value R -> 33R
- R22: renamed from R?; value R -> 82R
- RV2: renamed from RV?; value 1K -> 3K
- gave numbers to parts that had none: 58
Connections:
- net Earth: now also C5.2
- net at C8.1, Q3.3 (B), R15.1: now also Q1.3 (C); no longer Q2.3 (C)
- net at RV1.3: now also Q1.4 (E); no longer Q2.4 (E)
- net at R7.1, R8.2: now also Q1.5 (B); no longer Q2.5 (B)
- net at RV1.2: now also Q2.3 (C); no longer Q1.3 (C)
- net at C7.1, Q8.1 (E), R11.1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: now also Q2.1 (E); no longer Q2.1 (E)
- net at R4.1: now also Q2.2 (B); no longer Q2.2 (B)
- net at R3.2, R4.2: now also Q2.4 (E); no longer Q1.4 (E)
- net at C13.1, D1.2 (A), D2.1 (K)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: now also R23.1
- net at Q10.2 (B), R21.2: now also RV3.1; no longer R22.1
- net at Q11.2 (B): now also R24.1, RV4.3
- net at Q13.2 (D), R26.2: now also R24.2
- new net: Q2.5 (B), Q2.6 (C), R5.1
- new net: R22.1, RV3.2, RV3.3
- new net: R23.2, RV4.1, RV4.2
Other:
- moved on the sheet: C1, C10, C11, C12, C13, C2, C3, C4, C5, C6, C7, C8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

Commit message: Electric circuit Ver_1.2
Parts:
- R13: value 1K -> 470R
Other:
- moved on the sheet: C7, R10, R13, R6
Changed lines of the file:
@@
 L R R6
 U 1 1 5872933E
-P 3950 2750
-F 0 "R6" V 3850 2750 50  0000 C CNN
-F 1 "10K" V 3950 2750 50  0000 C CNN
-F 2 "" V 3880 2750 50  0000 C CNN
-F 3 "" H 3950 2750 50  0000 C CNN
-	1    3950 2750
+P 3950 2650
+F 0 "R6" V 3850 2650 50  0000 C CNN
+F 1 "10K" V 3950 2650 50  0000 C CNN
+F 2 "" V 3880 2650 50  0000 C CNN
+F 3 "" H 3950 2650 50  0000 C CNN
+	1    3950 2650
 	1    0    0    -1
 $EndComp
@@
 L Earth #PWR2
 U 1 1 587293F8
-P 3950 3000
-F 0 "#PWR2" H 3950 2750 50  0001 C CNN
-F 1 "Earth" H 3950 2850 50  0001 C CNN
-F 2 "" H 3950 3000 50  0000 C CNN
-F 3 "" H 3950 3000 50  0000 C CNN
-	1    3950 3000
+P 3950 2900
+F 0 "#PWR2" H 3950 2650 50  0001 C CNN
+F 1 "Earth" H 3950 2750 50  0001 C CNN
+F 2 "" H 3950 2900 50  0000 C CNN
+F 3 "" H 3950 2900 50  0000 C CNN
+	1    3950 2900
 	1    0    0    -1
 $EndComp
@@
 L CP1 C7
 U 1 1 58729487
-P 4400 1800
-F 0 "C7" H 4425 1900 50  0000 L CNN
-F 1 "47uF" H 4425 1700 50  0000 L CNN
-F 2 "" H 4400 1800 50  0000 C CNN
-F 3 "" H 4400 1800 50  0000 C CNN
-	1    4400 1800
+P 4400 1900
+F 0 "C7" H 4425 2000 50  0000 L CNN
+F 1 "47uF" H 4425 1800 50  0000 L CNN
+F 2 "" H 4400 1900 50  0000 C CNN
+F 3 "" H 4400 1900 50  0000 C CNN
+	1    4400 1900
 	1    0    0    -1
 $EndComp
@@
 L R R10
 U 1 1 5872B168
-P 4850 2900
-F 0 "R10" V 4750 2900 50  0000 C CNN
-F 1 "10K" V 4850 2900 50  0000 C CNN
-F 2 "" V 4780 2900 50  0000 C CNN
-F 3 "" H 4850 2900 50  0000 C CNN
-	1    4850 2900
+P 4850 2650
+F 0 "R10" V 4750 2650 50  0000 C CNN
+F 1 "10K" V 4850 2650 50  0000 C CNN
+F 2 "" V 4780 2650 50  0000 C CNN
+F 3 "" H 4850 2650 50  0000 C CNN
+	1    4850 2650
 	1    0    0    -1
 $EndComp
@@
 L R R13
 U 1 1 58733360
-P 5650 3900
-F 0 "R13" V 5550 3900 50  0000 C CNN
-F 1 "1K" V 5650 3900 50  0000 C CNN
-F 2 "" V 5580 3900 50  0000 C CNN
-F 3 "" H 5650 3900 50  0000 C CNN
-	1    5650 3900
+P 5650 3800
+F 0 "R13" V 5550 3800 50  0000 C CNN
+F 1 "470R" V 5650 3800 50  0000 C CNN
+F 2 "" V 5580 3800 50  0000 C CNN
+F 3 "" H 5650 3800 50  0000 C CNN
+	1    5650 3800
 	1    0    0    -1
 $EndComp
@@
 	3950 2350 3950 2450
 Wire Wire Line
-	3950 2450 3950 2600
-Wire Wire Line
-	4400 1500 4400 1650
+	3950 2450 3950 2500
+Wire Wire Line
+	4400 1500 4400 1750
 Connection ~ 3750 1500
 Wire Wire Line
-	4400 1950 4400 2450
+	4400 2050 4400 2450
 Wire Wire Line
 	4400 2450 3950 2450
@@
 	5250 2200 5350 2200
 Wire Wire Line
-	5250 2200 5250 2500
-Wire Wire Line
-	5250 2500 4850 2500
-Wire Wire Line
-	4850 2400 4850 2500
-Wire Wire Line
-	4850 2500 4850 2750
+	5250 2200 5250 2450
+Wire Wire Line
+	5250 2450 4850 2450
+Wire Wire Line
+	4850 2400 4850 2450
+Wire Wire Line
+	4850 2450 4850 2500
 Connection ~ 5250 2200
 Wire Wire Line
@@
 Wire Wire Line
 	3700 4050 3700 4000
-Connection ~ 4850 2500
-Wire Wire Line
-	4850 3050 4850 4500
+Connection ~ 4850 2450
+Wire Wire Line
+	4850 2800 4850 4500
 Wire Wire Line
 	4850 4500 4850 4600
@@
 Connection ~ 5650 4500
 Wire Wire Line
-	3950 2900 3950 3000
+	3950 2800 3950 2900
 Connection ~ 5650 1500
 Wire Wire Line
@@
 	5650 2850 5650 2900
 Wire Wire Line
-	5650 4050 5650 4250
+	5650 3950 5650 4250
 Wire Wire Line
 	5650 4250 5650 4500
@@
 	5650 3200 5650 3350
 Wire Wire Line
-	5650 3350 5650 3750
+	5650 3350 5650 3650
 Wire Wire Line
 	5500 3050 5500 3350

Commit message: Footprints Added
Parts:
- C1, C2: footprint (none) -> Capacitors_THT:C_Rect_L27_W9_H17_P23; Type Poly -> PP
- C10: footprint (none) -> Capacitors_THT:C_Rect_L7_W2.5_P5
- C11, C12: footprint (none) -> Capacitors_THT:C_Radial_D16_L31.5_P7.5
- C13: footprint (none) -> Capacitors_THT:C_Rect_L7_W2.5_P5; Type Poly -> PP
- C3: footprint (none) -> Capacitors_THT:C_Rect_L7_W4.5_P5
- C4, C5: footprint (none) -> Capacitors_THT:C_Rect_L7_W2.5_P5; Type (none) -> PP
- C6: footprint (none) -> Capacitors_THT:C_Radial_D13_L21_P5; Voltage 50V -> >=50V
- C7: footprint (none) -> Capacitors_THT:C_Radial_D10_L16_P5
- C8, C9: footprint (none) -> Capacitors_THT:C_Rect_L4_W2.5_P2.5
- D1, D2: value 15V -> 15V (1N4744A); footprint (none) -> Diodes_THT:Diode_DO-41_SOD81_Horizontal_RM10
- D3, D4: footprint (none) -> Diodes_THT:Diode_DO-35_SOD27_Horizontal_RM10
- F1, F2: footprint (none) -> Fuse_Holders_and_Fuses:Fuseholder5x20_horiz_SemiClosed_Casing10x25mm; Type (none) -> FX0321
- P1, P3: footprint (none) -> Connectors_Phoenix:PhoenixContact_MCV-G_02x3.81mm_Vertical
- P2, P4: footprint (none) -> Connectors:1pin
- Q1, Q2: footprint (none) -> TO_SOT_Packages_SMD:TSOT-6-MK06A_Handsoldering
- Q10, Q11: footprint (none) -> TO_SOT_Packages_THT:TO-92_Inline_Narrow_Oval
- Q12, Q13: footprint (none) -> TO_SOT_Packages_THT:TO-247_Vertical_Neutral123
- Q3, Q4, Q5, Q6, Q8, Q9: footprint (none) -> TO_SOT_Packages_THT:SOT126_SOT32_Housing_Vertical
- R1, R10, R11, R12, R13, R14, R15, R16, R17, R18, R19, R2, R20, R21, R22, R23, R24, R3, R4, R5, R6, R7, R8, R9: footprint (none) -> Resistors_THT:Resistor_Horizontal_RM10mm
- R25, R26: footprint (none) -> Resistors_THT:Resistor_Ceramic_Horizontal_L50mm-W14mm-H13mm-p60mm; Wattage 5W -> >=5W
- R27: footprint (none) -> Resistors_THT:Resistor_Ceramic_Horizontal_L19mm-W8mm-H8mm-p25mm
- RV1, RV2, RV3: footprint (none) -> Potentiometers:Potentiometer_Bourns_3296Y_3-8Zoll_Angular_ScrewUp; Type (none) -> Multi Turn
- RV4: value 50 -> 50R; footprint (none) -> Potentiometers:Potentiometer_Bourns_3296Y_3-8Zoll_Angular_ScrewUp; Type (none) -> Multi Turn

Commit message: Electric circuit Ver_1.3
Parts:
- added D1, D4: 1N4148, Diodes_THT:Diode_DO-35_SOD27_Horizontal_RM10, symbol D
- added P2, P3: TP, Connectors:1pin, symbol CONN_01X01
- D2: renamed from D1; value 15V (1N4744A) -> 15V
- D3: renamed from D2; value 15V (1N4744A) -> 15V
- renumbered D3 to D5, D4 to D6, P2 to P4, P3 to P5, P4 to P6
Connections:
- net at C10.1, Q5.2 (C), Q7.2 (C)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: now also D1.2 (A); no longer D2.1 (K)
- net at C8.2, Q3.2 (C), R10.2: now also P2.1 (P1)
- net at C10.2, C9.1, Q6.2 (C)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: now also D4.1 (K); no longer D3.2 (A)
- net at C13.1, D2.2 (A), D3.1 (K)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: now also P3.1 (P1)
- new net: D1.1 (K), D2.1 (K)
- new net: D3.2 (A), D4.2 (A)
Other:
- moved on the sheet: D2, D3

Commit message: Layout V1 added
Parts:
- Q7: footprint (none) -> TO_SOT_Packages_THT:SOT126_SOT32_Housing_Vertical
- RV3: value 50 -> 50R
Connections:
- net Earth: now also P1.1 (P1), P5.1 (P1), R1.1, R6.1; no longer P1.2 (P2), P5.2 (P2), R1.2, R6.2
- net at C1.1, C2.1: now also P1.2 (P2); no longer P1.1 (P1)
- net at C1.2, C2.2, R2.2: now also R1.2; no longer R1.1
- net at C7.1, Q2.1 (E), Q8.1 (E)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: now also R11.2, R9.2; no longer R11.1, R9.1
- net at Q1.5 (B), R8.2: now also R7.2; no longer R7.1
- net at C7.2, R5.2: now also R6.2; no longer R6.1
- net at Q4.1 (E): now also R9.1; no longer R9.2
- net at Q5.1 (E): now also R11.1; no longer R11.2
- net at C10.2, C9.1, D4.1 (K)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: now also R13.1; no longer R13.2
- net at C4.1, C5.1, C6.1: now also R7.1; no longer R7.2
- net at C13.1, D2.2 (A), D3.1 (K)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: now also P5.2 (P2), R26.2; no longer P5.1 (P1), R26.1
- net at F2.2, Q9.2 (C), R20.1: now also Q13.2 (D); no longer Q13.3 (S)
- net at RV2.1, RV2.2: now also R13.2; no longer R13.1
- net at Q11.2 (B), R24.1: now also RV4.1; no longer RV4.3
- net at R23.2, RV4.2: now also RV4.3; no longer RV4.1
- new net: Q13.3 (S), R24.2, R26.1
Changed lines of the file:
@@
 U 1 1 58727E75
 P 1150 3500
-F 0 "P1" H 1150 3650 50  0000 C CNN
-F 1 "Audio_In" H 1150 3350 50  0000 C CNN
+F 0 "P1" H 1150 3350 50  0000 C CNN
+F 1 "Audio_In" H 1150 3650 50  0000 C CNN
 F 2 "Connectors_Phoenix:PhoenixContact_MCV-G_02x3.81mm_Vertical" H 1150 3500 50  0001 C CNN
 F 3 "http://www.farnell.com/datasheets/2138215.pdf?_ga=1.58707370.1020810156.1482221903" H 1150 3500 50  0001 C CNN
 	1    1150 3500
-	-1   0    0    -1
+	-1   0    0    1
 $EndComp
 $Comp
@@
 F 3 "" H 1950 3650 50  0001 C CNN
 	1    1950 3650
-	1    0    0    -1
+	1    0    0    1
 $EndComp
 $Comp
@@
 $EndComp
 $Comp
-L Earth #PWR1
+L Earth #PWR01
 U 1 1 587282CB
 P 1400 3950
-F 0 "#PWR1" H 1400 3700 50  0001 C CNN
+F 0 "#PWR01" H 1400 3700 50  0001 C CNN
 F 1 "Earth" H 1400 3800 50  0001 C CNN
 F 2 "" H 1400 3950 50  0000 C CNN
@@
 F 3 "" H 3950 2650 50  0000 C CNN
 	1    3950 2650
-	1    0    0    -1
-$EndComp
-$Comp
-L Earth #PWR2
+	-1   0    0    1
+$EndComp
+$Comp
+L Earth #PWR02
 U 1 1 587293F8
 P 3950 2900
-F 0 "#PWR2" H 3950 2650 50  0001 C CNN
+F 0 "#PWR02" H 3950 2650 50  0001 C CNN
 F 1 "Earth" H 3950 2750 50  0001 C CNN
 F 2 "" H 3950 2900 50  0000 C CNN
@@
 F 3 "" H 4850 1750 50  0000 C CNN
 	1    4850 1750
-	1    0    0    -1
+	1    0    0    1
 $EndComp
 $Comp
@@
 F 3 "" H 5650 1750 50  0000 C CNN
 	1    5650 1750
-	1    0    0    -1
+	1    0    0    1
 $EndComp
 $Comp
@@
 F 3 "" H 3950 3700 50  0000 C CNN
 	1    3950 3700
-	1    0    0    -1
+	1    0    0    1
 $EndComp
 $Comp
@@
 $EndComp
 $Comp
-L Earth #PWR3
+L Earth #PWR03
 U 1 1 5872AAFE
 P 3950 4500
-F 0 "#PWR3" H 3950 4250 50  0001 C CNN
+F 0 "#PWR03" H 3950 4250 50  0001 C CNN
 F 1 "Earth" H 3950 4350 50  0001 C CNN
 F 2 "" H 3950 4500 50  0000 C CNN
@@
 U 1 1 5872E2CF
 P 9400 3500
-F 0 "P5" H 9400 3650 50  0000 C CNN
-F 1 "Audio_Out" H 9400 3350 50  0000 C CNN
+F 0 "P5" H 9400 3350 50  0000 C CNN
+F 1 "Audio_Out" H 9400 3650 50  0000 C CNN
 F 2 "Connectors_Phoenix:PhoenixContact_MCV-G_02x3.81mm_Vertical" H 9400 3500 50  0001 C CNN
 F 3 "" H 9400 3500 50  0000 C CNN
 	1    9400 3500
-	1    0    0    -1
-$EndComp
-$Comp
-L Earth #PWR7
+	1    0    0    1
+$EndComp
+$Comp
+L Earth #PWR04
 U 1 1 5872EA23
 P 9100 3900
-F 0 "#PWR7" H 9100 3650 50  0001 C CNN
+F 0 "#PWR04" H 9100 3650 50  0001 C CNN
 F 1 "Earth" H 9100 3750 50  0001 C CNN
 F 2 "" H 9100 3900 50  0000 C CNN
@@
 $EndComp
 $Comp
-L Earth #PWR6
+L Earth #PWR05
 U 1 1 5872FA97
 P 8850 4350
-F 0 "#PWR6" H 8850 4100 50  0001 C CNN
+F 0 "#PWR05" H 8850 4100 50  0001 C CNN
 F 1 "Earth" H 8850 4200 50  0001 C CNN
 F 2 "" H 8850 4350 50  0000 C CNN
@@
 F 3 "" H 5650 3800 50  0000 C CNN
 	1    5650 3800
-	1    0    0    -1
+	1    0    0    1
 $EndComp
 $Comp
@@
 F 0 "Q7" H 6150 2925 50  0000 L CNN
 F 1 "BD139" H 6150 2850 50  0000 L CNN
-F 2 "" H 6150 2775 50  0000 L CIN
+F 2 "TO_SOT_Packages_THT:SOT126_SOT32_Housing_Vertical" H 6150 2775 50  0001 L CIN
 F 3 "" H 5950 2850 50  0000 L CNN
 	1    5950 2850
@@
 F 4 ">=5W" V 8500 4050 60  0001 C CNN "Wattage"
 	1    8500 4050
-	1    0    0    -1
+	1    0    0    1
 $EndComp
 $Comp
@@
 F 3 "" H 8400 4850 50  0000 C CNN
 	1    8400 4850
-	1    0    0    -1
+	1    0    0    1
 $EndComp
 $Comp
@@
 $EndComp
 $Comp
-L Earth #PWR4
+L Earth #PWR06
 U 1 1 5875481E
 P 7150 2250
-F 0 "#PWR4" H 7150 2000 50  0001 C CNN
+F 0 "#PWR06" H 7150 2000 50  0001 C CNN
 F 1 "Earth" H 7150 2100 50  0001 C CNN
 F 2 "" H 7150 2250 50  0000 C CNN
@@
 $EndComp
 $Comp
-L Earth #PWR5
+L Earth #PWR07
 U 1 1 587571E8
 P 7150 6200
-F 0 "#PWR5" H 7150 5950 50  0001 C CNN
+F 0 "#PWR07" H 7150 5950 50  0001 C CNN
 F 1 "Earth" H 7150 6050 50  0001 C CNN
 F 2 "" H 7150 6200 50  0000 C CNN
@@
 P 8100 2850
 F 0 "RV3" V 7925 2850 50  0000 C CNN
-F 1 "50" V 8000 2850 50  0000 C CNN
+F 1 "50R" V 8000 2850 50  0000 C CNN
 F 2 "Potentiometers:Potentiometer_Bourns_3296Y_3-8Zoll_Angular_ScrewUp" H 8100 2850 50  0001 C CNN
 F 3 "http://www.farnell.com/datasheets/2061261.pdf?_ga=1.94292381.1020810156.1482221903" H 8100 2850 50  0001 C CNN
@@
 F 4 "Multi Turn" V 8100 4050 60  0001 C CNN "Type"
 	1    8100 4050
-	1    0    0    -1
+	1    0    0    1
 $EndComp
 Wire Wire Line

Commit message: Layout V1.1 + routing V1
Parts:
- added P7: TP, Connectors:1pin, symbol CONN_01X01
- renumbered Q2 to Q1, Q1 to Q2
Connections:
- net Earth: now also P7.1 (P1)
- net at Q2.6 (C), R5.1: now also Q2.5 (B); no longer Q1.5 (B)
- net at RV1.2: now also Q2.3 (C); no longer Q1.3 (C)
- net at RV1.3: now also Q1.4 (E); no longer Q2.4 (E)
- net at R3.2, R4.2: now also Q2.4 (E); no longer Q1.4 (E)
- net at C8.1, Q3.3 (B), R15.1: now also Q1.3 (C); no longer Q2.3 (C)
- net at R7.2, R8.2: now also Q1.5 (B); no longer Q2.5 (B)
Other:
- moved on the sheet: Q1B, Q2B
